Commit message: change uav dynamics

File: assets/quadrotor.urdf (robot description, URDF)
Before this commit: robot simple_quadrotor, 5 links, 4 joints
Links:
- removed link rotor_0
- removed link rotor_1
- removed link rotor_2
- removed link rotor_3
- added link center_of_mass_link, mass 0
- added link prop0_link, mass 0
- added link prop1_link, mass 0
- added link prop2_link, mass 0
- added link prop3_link, mass 0
- link base_link: mass 0.03 -> 0.027; geometry collision cylinder length=.025 radius=.06; visual box size=0.06 0.06 0.02
Joints:
- removed joint joint_rotor_0
- removed joint joint_rotor_1
- removed joint joint_rotor_2
- removed joint joint_rotor_3
- added joint center_of_mass_joint: type fixed, parent base_link, child center_of_mass_link
- added joint prop0_joint: type fixed, parent base_link, child prop0_link
- added joint prop1_joint: type fixed, parent base_link, child prop1_link
- added joint prop2_joint: type fixed, parent base_link, child prop2_link
- added joint prop3_joint: type fixed, parent base_link, child prop3_link

Commit message: path planning v1

File: assets/quadrotor.urdf (robot description, URDF)
Before this commit: robot cf2, 6 links, 5 joints
Links:
- link prop0_link: geometry visual cylinder length=0.002 radius=0.023
- link prop1_link: geometry visual cylinder length=0.002 radius=0.023
- link prop2_link: geometry visual cylinder length=0.002 radius=0.023
- link prop3_link: geometry visual cylinder length=0.002 radius=0.023

Commit message: change urdf

File: assets/quadrotor.urdf (robot description, URDF)
Before this commit: robot cf2, 6 links, 5 joints
Links:
- link base_link: geometry collision box size=0.15 0.15 0.06; visual box size=0.1 0.1 0.05
- link prop0_link: geometry visual cylinder length=0.002 radius=0.05
- link prop1_link: geometry visual cylinder length=0.002 radius=0.05
- link prop2_link: geometry visual cylinder length=0.002 radius=0.05
- link prop3_link: geometry visual cylinder length=0.002 radius=0.05
