Commit message: Debug et modification pour code plus robuste et ajout de features

File: assets/city.urdf (robot description, URDF)
Before this commit: robot city, 146 links, 145 joints
Links:
- link bld_1: geometry collision box size=6.0 6.0 44.4; visual box size=6.0 6.0 44.4
- link bld_10: geometry collision box size=6.0 6.0 41.8; visual box size=6.0 6.0 41.8
- link bld_100: geometry collision box size=6.0 6.0 43.9; visual box size=6.0 6.0 43.9
- link bld_101: geometry collision box size=6.0 6.0 33.5; visual box size=6.0 6.0 33.5
- link bld_102: geometry collision box size=6.0 6.0 42.0; visual box size=6.0 6.0 42.0
- link bld_103: geometry collision box size=6.0 6.0 48.6; visual box size=6.0 6.0 48.6
- link bld_104: geometry collision box size=6.0 6.0 31.1; visual box size=6.0 6.0 31.1
- link bld_105: geometry collision box size=6.0 6.0 48.9; visual box size=6.0 6.0 48.9
- link bld_106: geometry collision box size=6.0 6.0 46.2; visual box size=6.0 6.0 46.2
- link bld_107: geometry collision box size=6.0 6.0 33.5; visual box size=6.0 6.0 33.5
- link bld_108: geometry collision box size=6.0 6.0 46.5; visual box size=6.0 6.0 46.5
- link bld_109: geometry collision box size=6.0 6.0 40.2; visual box size=6.0 6.0 40.2
- link bld_11: geometry collision box size=6.0 6.0 43.4; visual box size=6.0 6.0 43.4
- link bld_110: geometry collision box size=6.0 6.0 39.6; visual box size=6.0 6.0 39.6
- link bld_111: geometry collision box size=6.0 6.0 46.4; visual box size=6.0 6.0 46.4
- link bld_112: geometry collision box size=6.0 6.0 46.3; visual box size=6.0 6.0 46.3
- link bld_113: geometry collision box size=6.0 6.0 36.0; visual box size=6.0 6.0 36.0
- link bld_114: geometry collision box size=6.0 6.0 37.9; visual box size=6.0 6.0 37.9
- link bld_115: geometry collision box size=6.0 6.0 45.4; visual box size=6.0 6.0 45.4
- link bld_116: geometry collision box size=6.0 6.0 47.1; visual box size=6.0 6.0 47.1
- link bld_117: geometry collision box size=6.0 6.0 49.3; visual box size=6.0 6.0 49.3
- link bld_118: geometry collision box size=6.0 6.0 37.7; visual box size=6.0 6.0 37.7
- link bld_119: geometry collision box size=6.0 6.0 44.5; visual box size=6.0 6.0 44.5
- link bld_12: geometry collision box size=6.0 6.0 49.5; visual box size=6.0 6.0 49.5
- link bld_120: geometry collision box size=6.0 6.0 35.9; visual box size=6.0 6.0 35.9
- link bld_121: geometry collision box size=6.0 6.0 45.2; visual box size=6.0 6.0 45.2
- link bld_122: geometry collision box size=6.0 6.0 44.3; visual box size=6.0 6.0 44.3
- link bld_123: geometry collision box size=6.0 6.0 47.2; visual box size=6.0 6.0 47.2
- link bld_124: geometry collision box size=6.0 6.0 38.2; visual box size=6.0 6.0 38.2
- link bld_125: geometry collision box size=6.0 6.0 33.9; visual box size=6.0 6.0 33.9
- link bld_126: geometry collision box size=6.0 6.0 30.9; visual box size=6.0 6.0 30.9
- link bld_127: geometry collision box size=6.0 6.0 36.6; visual box size=6.0 6.0 36.6
- link bld_128: geometry collision box size=6.0 6.0 35.8; visual box size=6.0 6.0 35.8
- link bld_129: geometry collision box size=6.0 6.0 40.7; visual box size=6.0 6.0 40.7
- link bld_13: geometry collision box size=6.0 6.0 36.7; visual box size=6.0 6.0 36.7
- link bld_130: geometry collision box size=6.0 6.0 33.9; visual box size=6.0 6.0 33.9
- link bld_131: geometry collision box size=6.0 6.0 30.5; visual box size=6.0 6.0 30.5
- link bld_132: geometry collision box size=6.0 6.0 45.7; visual box size=6.0 6.0 45.7
- link bld_133: geometry collision box size=6.0 6.0 31.0; visual box size=6.0 6.0 31.0
- link bld_134: geometry collision box size=6.0 6.0 41.4; visual box size=6.0 6.0 41.4
- link bld_135: geometry collision box size=6.0 6.0 43.6; visual box size=6.0 6.0 43.6
- link bld_136: geometry collision box size=6.0 6.0 35.6; visual box size=6.0 6.0 35.6
- link bld_137: geometry collision box size=6.0 6.0 46.6; visual box size=6.0 6.0 46.6
- link bld_138: geometry collision box size=6.0 6.0 30.1; visual box size=6.0 6.0 30.1
- link bld_139: geometry collision box size=6.0 6.0 42.4; visual box size=6.0 6.0 42.4
- link bld_14: geometry collision box size=6.0 6.0 32.1; visual box size=6.0 6.0 32.1
- link bld_140: geometry collision box size=6.0 6.0 49.3; visual box size=6.0 6.0 49.3
- link bld_141: geometry collision box size=6.0 6.0 34.6; visual box size=6.0 6.0 34.6
- link bld_142: geometry collision box size=6.0 6.0 45.7; visual box size=6.0 6.0 45.7
- link bld_143: geometry collision box size=6.0 6.0 32.0; visual box size=6.0 6.0 32.0
- link bld_15: geometry collision box size=6.0 6.0 47.5; visual box size=6.0 6.0 47.5
- link bld_16: geometry collision box size=6.0 6.0 38.6; visual box size=6.0 6.0 38.6
- link bld_17: geometry collision box size=6.0 6.0 32.3; visual box size=6.0 6.0 32.3
- link bld_18: geometry collision box size=6.0 6.0 42.2; visual box size=6.0 6.0 42.2
- link bld_19: geometry collision box size=6.0 6.0 37.3; visual box size=6.0 6.0 37.3
- link bld_2: geometry collision box size=6.0 6.0 32.1; visual box size=6.0 6.0 32.1
- link bld_20: geometry collision box size=6.0 6.0 49.4; visual box size=6.0 6.0 49.4
- link bld_21: geometry collision box size=6.0 6.0 39.5; visual box size=6.0 6.0 39.5
- link bld_22: geometry collision box size=6.0 6.0 35.3; visual box size=6.0 6.0 35.3
- link bld_23: geometry collision box size=6.0 6.0 35.1; visual box size=6.0 6.0 35.1
- link bld_24: geometry collision box size=6.0 6.0 49.1; visual box size=6.0 6.0 49.1
- link bld_25: geometry collision box size=6.0 6.0 35.9; visual box size=6.0 6.0 35.9
- link bld_26: geometry collision box size=6.0 6.0 33.3; visual box size=6.0 6.0 33.3
- link bld_27: geometry collision box size=6.0 6.0 47.7; visual box size=6.0 6.0 47.7
- link bld_28: geometry collision box size=6.0 6.0 32.5; visual box size=6.0 6.0 32.5
- link bld_29: geometry collision box size=6.0 6.0 45.8; visual box size=6.0 6.0 45.8
- link bld_3: geometry collision box size=6.0 6.0 42.3; visual box size=6.0 6.0 42.3
- link bld_30: geometry collision box size=6.0 6.0 41.8; visual box size=6.0 6.0 41.8
- link bld_31: geometry collision box size=6.0 6.0 37.7; visual box size=6.0 6.0 37.7
- link bld_32: geometry collision box size=6.0 6.0 46.9; visual box size=6.0 6.0 46.9
- link bld_33: geometry collision box size=6.0 6.0 35.3; visual box size=6.0 6.0 35.3
- link bld_34: geometry collision box size=6.0 6.0 37.8; visual box size=6.0 6.0 37.8
- link bld_35: geometry collision box size=6.0 6.0 47.4; visual box size=6.0 6.0 47.4
- link bld_36: geometry collision box size=6.0 6.0 42.5; visual box size=6.0 6.0 42.5
- link bld_37: geometry collision box size=6.0 6.0 34.8; visual box size=6.0 6.0 34.8
- link bld_38: geometry collision box size=6.0 6.0 34.2; visual box size=6.0 6.0 34.2
- link bld_39: geometry collision box size=6.0 6.0 39.8; visual box size=6.0 6.0 39.8
- link bld_4: geometry collision box size=6.0 6.0 30.8; visual box size=6.0 6.0 30.8
- link bld_40: geometry collision box size=6.0 6.0 43.2; visual box size=6.0 6.0 43.2
- link bld_41: geometry collision box size=6.0 6.0 36.5; visual box size=6.0 6.0 36.5
- link bld_42: geometry collision box size=6.0 6.0 43.7; visual box size=6.0 6.0 43.7
- link bld_43: geometry collision box size=6.0 6.0 38.4; visual box size=6.0 6.0 38.4
- link bld_44: geometry collision box size=6.0 6.0 38.7; visual box size=6.0 6.0 38.7
- link bld_45: geometry collision box size=6.0 6.0 43.9; visual box size=6.0 6.0 43.9
- link bld_46: geometry collision box size=6.0 6.0 43.2; visual box size=6.0 6.0 43.2
- link bld_47: geometry collision box size=6.0 6.0 38.7; visual box size=6.0 6.0 38.7
- link bld_48: geometry collision box size=6.0 6.0 39.2; visual box size=6.0 6.0 39.2
- link bld_49: geometry collision box size=6.0 6.0 45.3; visual box size=6.0 6.0 45.3
- link bld_5: geometry collision box size=6.0 6.0 46.1; visual box size=6.0 6.0 46.1
- link bld_50: geometry collision box size=6.0 6.0 32.9; visual box size=6.0 6.0 32.9
- link bld_51: geometry collision box size=6.0 6.0 38.1; visual box size=6.0 6.0 38.1
- link bld_52: geometry collision box size=6.0 6.0 48.3; visual box size=6.0 6.0 48.3
- link bld_53: geometry collision box size=6.0 6.0 37.1; visual box size=6.0 6.0 37.1
- link bld_54: geometry collision box size=6.0 6.0 30.9; visual box size=6.0 6.0 30.9
- link bld_55: geometry collision box size=6.0 6.0 49.7; visual box size=6.0 6.0 49.7
- link bld_56: geometry collision box size=6.0 6.0 30.8; visual box size=6.0 6.0 30.8
- link bld_57: geometry collision box size=6.0 6.0 45.1; visual box size=6.0 6.0 45.1
- link bld_58: geometry collision box size=6.0 6.0 40.2; visual box size=6.0 6.0 40.2
- link bld_59: geometry collision box size=6.0 6.0 38.4; visual box size=6.0 6.0 38.4
- link bld_6: geometry collision box size=6.0 6.0 42.1; visual box size=6.0 6.0 42.1
- link bld_60: geometry collision box size=6.0 6.0 37.4; visual box size=6.0 6.0 37.4
- link bld_61: geometry collision box size=6.0 6.0 44.2; visual box size=6.0 6.0 44.2
- link bld_62: geometry collision box size=6.0 6.0 35.8; visual box size=6.0 6.0 35.8
- link bld_63: geometry collision box size=6.0 6.0 40.4; visual box size=6.0 6.0 40.4
- link bld_64: geometry collision box size=6.0 6.0 32.3; visual box size=6.0 6.0 32.3
- link bld_65: geometry collision box size=6.0 6.0 41.6; visual box size=6.0 6.0 41.6
- link bld_66: geometry collision box size=6.0 6.0 31.6; visual box size=6.0 6.0 31.6
- link bld_67: geometry collision box size=6.0 6.0 44.2; visual box size=6.0 6.0 44.2
- link bld_68: geometry collision box size=6.0 6.0 47.3; visual box size=6.0 6.0 47.3
- link bld_69: geometry collision box size=6.0 6.0 41.5; visual box size=6.0 6.0 41.5
- link bld_7: geometry collision box size=6.0 6.0 37.6; visual box size=6.0 6.0 37.6
- link bld_70: geometry collision box size=6.0 6.0 36.8; visual box size=6.0 6.0 36.8
- link bld_71: geometry collision box size=6.0 6.0 46.4; visual box size=6.0 6.0 46.4
- link bld_72: geometry collision box size=6.0 6.0 44.6; visual box size=6.0 6.0 44.6
- link bld_73: geometry collision box size=6.0 6.0 30.9; visual box size=6.0 6.0 30.9
- link bld_74: geometry collision box size=6.0 6.0 46.4; visual box size=6.0 6.0 46.4
- link bld_75: geometry collision box size=6.0 6.0 46.4; visual box size=6.0 6.0 46.4
- link bld_76: geometry collision box size=6.0 6.0 42.9; visual box size=6.0 6.0 42.9
- link bld_77: geometry collision box size=6.0 6.0 43.7; visual box size=6.0 6.0 43.7
- link bld_78: geometry collision box size=6.0 6.0 40.6; visual box size=6.0 6.0 40.6
- link bld_79: geometry collision box size=6.0 6.0 35.8; visual box size=6.0 6.0 35.8
- link bld_8: geometry collision box size=6.0 6.0 30.8; visual box size=6.0 6.0 30.8
- link bld_80: geometry collision box size=6.0 6.0 43.1; visual box size=6.0 6.0 43.1
- link bld_81: geometry collision box size=6.0 6.0 48.9; visual box size=6.0 6.0 48.9
- link bld_82: geometry collision box size=6.0 6.0 36.7; visual box size=6.0 6.0 36.7
- link bld_83: geometry collision box size=6.0 6.0 36.9; visual box size=6.0 6.0 36.9
- link bld_84: geometry collision box size=6.0 6.0 37.0; visual box size=6.0 6.0 37.0
- link bld_85: geometry collision box size=6.0 6.0 45.8; visual box size=6.0 6.0 45.8
- link bld_86: geometry collision box size=6.0 6.0 34.5; visual box size=6.0 6.0 34.5
- link bld_87: geometry collision box size=6.0 6.0 46.5; visual box size=6.0 6.0 46.5
- link bld_88: geometry collision box size=6.0 6.0 45.9; visual box size=6.0 6.0 45.9
- link bld_89: geometry collision box size=6.0 6.0 31.2; visual box size=6.0 6.0 31.2
- link bld_9: geometry collision box size=6.0 6.0 46.7; visual box size=6.0 6.0 46.7
- link bld_90: geometry collision box size=6.0 6.0 37.2; visual box size=6.0 6.0 37.2
- link bld_91: geometry collision box size=6.0 6.0 34.8; visual box size=6.0 6.0 34.8
- link bld_92: geometry collision box size=6.0 6.0 33.2; visual box size=6.0 6.0 33.2
- link bld_93: geometry collision box size=6.0 6.0 45.7; visual box size=6.0 6.0 45.7
- link bld_94: geometry collision box size=6.0 6.0 44.1; visual box size=6.0 6.0 44.1
- link bld_95: geometry collision box size=6.0 6.0 39.0; visual box size=6.0 6.0 39.0
- link bld_96: geometry collision box size=6.0 6.0 36.9; visual box size=6.0 6.0 36.9
- link bld_97: geometry collision box size=6.0 6.0 48.9; visual box size=6.0 6.0 48.9
- link bld_98: geometry collision box size=6.0 6.0 35.4; visual box size=6.0 6.0 35.4
- link bld_99: geometry collision box size=6.0 6.0 46.0; visual box size=6.0 6.0 46.0
Joints:
- joint j_bld_1: origin xyz=-51.666666666666664 -45.0 23.0 rpy=0 0 0 -> xyz=-51.666666666666664 -45.0 22.2 rpy=0 0 0
- joint j_bld_10: origin xyz=-51.666666666666664 -15.0 20.15 rpy=0 0 0 -> xyz=-51.666666666666664 -15.0 20.9 rpy=0 0 0
- joint j_bld_100: origin xyz=8.333333333333334 45.0 24.25 rpy=0 0 0 -> xyz=8.333333333333334 45.0 21.95 rpy=0 0 0
- joint j_bld_101: origin xyz=8.333333333333334 51.666666666666664 24.9 rpy=0 0 0 -> xyz=8.333333333333334 51.666666666666664 16.75 rpy=0 0 0
- joint j_bld_102: origin xyz=15.0 38.333333333333336 22.8 rpy=0 0 0 -> xyz=15.0 38.333333333333336 21.0 rpy=0 0 0
- joint j_bld_103: origin xyz=15.0 45.0 24.45 rpy=0 0 0 -> xyz=15.0 45.0 24.3 rpy=0 0 0
- joint j_bld_104: origin xyz=15.0 51.666666666666664 23.1 rpy=0 0 0 -> xyz=15.0 51.666666666666664 15.55 rpy=0 0 0
- joint j_bld_105: origin xyz=21.666666666666668 38.333333333333336 16.75 rpy=0 0 0 -> xyz=21.666666666666668 38.333333333333336 24.45 rpy=0 0 0
- joint j_bld_106: origin xyz=21.666666666666668 45.0 17.55 rpy=0 0 0 -> xyz=21.666666666666668 45.0 23.1 rpy=0 0 0
- joint j_bld_107: origin xyz=21.666666666666668 51.666666666666664 18.9 rpy=0 0 0 -> xyz=21.666666666666668 51.666666666666664 16.75 rpy=0 0 0
- joint j_bld_108: origin xyz=38.333333333333336 -51.666666666666664 15.9 rpy=0 0 0 -> xyz=38.333333333333336 -51.666666666666664 23.25 rpy=0 0 0
- joint j_bld_109: origin xyz=38.333333333333336 -45.0 18.75 rpy=0 0 0 -> xyz=38.333333333333336 -45.0 20.1 rpy=0 0 0
- joint j_bld_11: origin xyz=-51.666666666666664 -8.333333333333332 22.4 rpy=0 0 0 -> xyz=-51.666666666666664 -8.333333333333332 21.7 rpy=0 0 0
- joint j_bld_110: origin xyz=38.333333333333336 -38.333333333333336 17.2 rpy=0 0 0 -> xyz=38.333333333333336 -38.333333333333336 19.8 rpy=0 0 0
- joint j_bld_111: origin xyz=45.0 -51.666666666666664 16.15 rpy=0 0 0 -> xyz=45.0 -51.666666666666664 23.2 rpy=0 0 0
- joint j_bld_112: origin xyz=45.0 -45.0 21.75 rpy=0 0 0 -> xyz=45.0 -45.0 23.15 rpy=0 0 0
- joint j_bld_113: origin xyz=45.0 -38.333333333333336 23.6 rpy=0 0 0 -> xyz=45.0 -38.333333333333336 18.0 rpy=0 0 0
- joint j_bld_114: origin xyz=51.666666666666664 -51.666666666666664 24.95 rpy=0 0 0 -> xyz=51.666666666666664 -51.666666666666664 18.95 rpy=0 0 0
- joint j_bld_115: origin xyz=51.666666666666664 -45.0 22.4 rpy=0 0 0 -> xyz=51.666666666666664 -45.0 22.7 rpy=0 0 0
- joint j_bld_116: origin xyz=51.666666666666664 -38.333333333333336 22.45 rpy=0 0 0 -> xyz=51.666666666666664 -38.333333333333336 23.55 rpy=0 0 0
- joint j_bld_117: origin xyz=38.333333333333336 -21.666666666666664 23.75 rpy=0 0 0 -> xyz=38.333333333333336 -21.666666666666664 24.65 rpy=0 0 0
- joint j_bld_118: origin xyz=38.333333333333336 -15.0 15.5 rpy=0 0 0 -> xyz=38.333333333333336 -15.0 18.85 rpy=0 0 0
- joint j_bld_119: origin xyz=38.333333333333336 -8.333333333333332 24.75 rpy=0 0 0 -> xyz=38.333333333333336 -8.333333333333332 22.25 rpy=0 0 0
- joint j_bld_12: origin xyz=-45.0 -21.666666666666664 21.65 rpy=0 0 0 -> xyz=-45.0 -21.666666666666664 24.75 rpy=0 0 0
- joint j_bld_120: origin xyz=45.0 -21.666666666666664 22.25 rpy=0 0 0 -> xyz=45.0 -21.666666666666664 17.95 rpy=0 0 0
- joint j_bld_121: origin xyz=45.0 -15.0 24.15 rpy=0 0 0 -> xyz=45.0 -15.0 22.6 rpy=0 0 0
- joint j_bld_122: origin xyz=45.0 -8.333333333333332 24.7 rpy=0 0 0 -> xyz=45.0 -8.333333333333332 22.15 rpy=0 0 0
- joint j_bld_123: origin xyz=51.666666666666664 -21.666666666666664 24.1 rpy=0 0 0 -> xyz=51.666666666666664 -21.666666666666664 23.6 rpy=0 0 0
- joint j_bld_124: origin xyz=51.666666666666664 -15.0 19.95 rpy=0 0 0 -> xyz=51.666666666666664 -15.0 19.1 rpy=0 0 0
- joint j_bld_125: origin xyz=51.666666666666664 -8.333333333333332 22.6 rpy=0 0 0 -> xyz=51.666666666666664 -8.333333333333332 16.95 rpy=0 0 0
- joint j_bld_126: origin xyz=38.333333333333336 8.333333333333334 18.9 rpy=0 0 0 -> xyz=38.333333333333336 8.333333333333334 15.45 rpy=0 0 0
- joint j_bld_127: origin xyz=38.333333333333336 15.0 19.9 rpy=0 0 0 -> xyz=38.333333333333336 15.0 18.3 rpy=0 0 0
- joint j_bld_128: origin xyz=38.333333333333336 21.666666666666668 17.1 rpy=0 0 0 -> xyz=38.333333333333336 21.666666666666668 17.9 rpy=0 0 0
- joint j_bld_129: origin xyz=45.0 8.333333333333334 21.2 rpy=0 0 0 -> xyz=45.0 8.333333333333334 20.35 rpy=0 0 0
- joint j_bld_13: origin xyz=-45.0 -15.0 19.3 rpy=0 0 0 -> xyz=-45.0 -15.0 18.35 rpy=0 0 0
- joint j_bld_130: origin xyz=45.0 15.0 17.75 rpy=0 0 0 -> xyz=45.0 15.0 16.95 rpy=0 0 0
- joint j_bld_131: origin xyz=45.0 21.666666666666668 22.1 rpy=0 0 0 -> xyz=45.0 21.666666666666668 15.25 rpy=0 0 0
- joint j_bld_132: origin xyz=51.666666666666664 8.333333333333334 16.55 rpy=0 0 0 -> xyz=51.666666666666664 8.333333333333334 22.85 rpy=0 0 0
- joint j_bld_133: origin xyz=51.666666666666664 15.0 24.0 rpy=0 0 0 -> xyz=51.666666666666664 15.0 15.5 rpy=0 0 0
- joint j_bld_134: origin xyz=51.666666666666664 21.666666666666668 24.9 rpy=0 0 0 -> xyz=51.666666666666664 21.666666666666668 20.7 rpy=0 0 0
- joint j_bld_135: origin xyz=38.333333333333336 38.333333333333336 19.4 rpy=0 0 0 -> xyz=38.333333333333336 38.333333333333336 21.8 rpy=0 0 0
- joint j_bld_136: origin xyz=38.333333333333336 45.0 24.75 rpy=0 0 0 -> xyz=38.333333333333336 45.0 17.8 rpy=0 0 0
- joint j_bld_137: origin xyz=38.333333333333336 51.666666666666664 24.0 rpy=0 0 0 -> xyz=38.333333333333336 51.666666666666664 23.3 rpy=0 0 0
- joint j_bld_138: origin xyz=45.0 38.333333333333336 18.9 rpy=0 0 0 -> xyz=45.0 38.333333333333336 15.05 rpy=0 0 0
- joint j_bld_139: origin xyz=45.0 45.0 24.7 rpy=0 0 0 -> xyz=45.0 45.0 21.2 rpy=0 0 0
- joint j_bld_14: origin xyz=-45.0 -8.333333333333332 24.6 rpy=0 0 0 -> xyz=-45.0 -8.333333333333332 16.05 rpy=0 0 0
- joint j_bld_140: origin xyz=45.0 51.666666666666664 19.35 rpy=0 0 0 -> xyz=45.0 51.666666666666664 24.65 rpy=0 0 0
- joint j_bld_141: origin xyz=51.666666666666664 38.333333333333336 23.55 rpy=0 0 0 -> xyz=51.666666666666664 38.333333333333336 17.3 rpy=0 0 0
- joint j_bld_142: origin xyz=51.666666666666664 45.0 21.9 rpy=0 0 0 -> xyz=51.666666666666664 45.0 22.85 rpy=0 0 0
- joint j_bld_143: origin xyz=51.666666666666664 51.666666666666664 22.6 rpy=0 0 0 -> xyz=51.666666666666664 51.666666666666664 16.0 rpy=0 0 0
- joint j_bld_15: origin xyz=-38.333333333333336 -21.666666666666664 16.95 rpy=0 0 0 -> xyz=-38.333333333333336 -21.666666666666664 23.75 rpy=0 0 0
- joint j_bld_16: origin xyz=-38.333333333333336 -15.0 18.45 rpy=0 0 0 -> xyz=-38.333333333333336 -15.0 19.3 rpy=0 0 0
- joint j_bld_17: origin xyz=-38.333333333333336 -8.333333333333332 24.65 rpy=0 0 0 -> xyz=-38.333333333333336 -8.333333333333332 16.15 rpy=0 0 0
- joint j_bld_18: origin xyz=-51.666666666666664 8.333333333333334 22.05 rpy=0 0 0 -> xyz=-51.666666666666664 8.333333333333334 21.1 rpy=0 0 0
- joint j_bld_19: origin xyz=-51.666666666666664 15.0 23.2 rpy=0 0 0 -> xyz=-51.666666666666664 15.0 18.65 rpy=0 0 0
- joint j_bld_2: origin xyz=-51.666666666666664 -38.333333333333336 18.65 rpy=0 0 0 -> xyz=-51.666666666666664 -38.333333333333336 16.05 rpy=0 0 0
- joint j_bld_20: origin xyz=-51.666666666666664 21.666666666666668 19.15 rpy=0 0 0 -> xyz=-51.666666666666664 21.666666666666668 24.7 rpy=0 0 0
- joint j_bld_21: origin xyz=-45.0 8.333333333333334 20.2 rpy=0 0 0 -> xyz=-45.0 8.333333333333334 19.75 rpy=0 0 0
- joint j_bld_22: origin xyz=-45.0 15.0 22.95 rpy=0 0 0 -> xyz=-45.0 15.0 17.65 rpy=0 0 0
- joint j_bld_23: origin xyz=-45.0 21.666666666666668 20.15 rpy=0 0 0 -> xyz=-45.0 21.666666666666668 17.55 rpy=0 0 0
- joint j_bld_24: origin xyz=-38.333333333333336 8.333333333333334 15.45 rpy=0 0 0 -> xyz=-38.333333333333336 8.333333333333334 24.55 rpy=0 0 0
- joint j_bld_25: origin xyz=-38.333333333333336 15.0 24.95 rpy=0 0 0 -> xyz=-38.333333333333336 15.0 17.95 rpy=0 0 0
- joint j_bld_26: origin xyz=-38.333333333333336 21.666666666666668 23.4 rpy=0 0 0 -> xyz=-38.333333333333336 21.666666666666668 16.65 rpy=0 0 0
- joint j_bld_27: origin xyz=-51.666666666666664 38.333333333333336 22.35 rpy=0 0 0 -> xyz=-51.666666666666664 38.333333333333336 23.85 rpy=0 0 0
- joint j_bld_28: origin xyz=-51.666666666666664 45.0 19.5 rpy=0 0 0 -> xyz=-51.666666666666664 45.0 16.25 rpy=0 0 0
- joint j_bld_29: origin xyz=-51.666666666666664 51.666666666666664 20.8 rpy=0 0 0 -> xyz=-51.666666666666664 51.666666666666664 22.9 rpy=0 0 0
- joint j_bld_3: origin xyz=-45.0 -51.666666666666664 19.4 rpy=0 0 0 -> xyz=-45.0 -51.666666666666664 21.15 rpy=0 0 0
- joint j_bld_30: origin xyz=-45.0 38.333333333333336 21.7 rpy=0 0 0 -> xyz=-45.0 38.333333333333336 20.9 rpy=0 0 0
- joint j_bld_31: origin xyz=-45.0 45.0 21.4 rpy=0 0 0 -> xyz=-45.0 45.0 18.85 rpy=0 0 0
- joint j_bld_32: origin xyz=-45.0 51.666666666666664 21.2 rpy=0 0 0 -> xyz=-45.0 51.666666666666664 23.45 rpy=0 0 0
- joint j_bld_33: origin xyz=-38.333333333333336 38.333333333333336 20.4 rpy=0 0 0 -> xyz=-38.333333333333336 38.333333333333336 17.65 rpy=0 0 0
- joint j_bld_34: origin xyz=-38.333333333333336 45.0 16.55 rpy=0 0 0 -> xyz=-38.333333333333336 45.0 18.9 rpy=0 0 0
- joint j_bld_35: origin xyz=-38.333333333333336 51.666666666666664 22.15 rpy=0 0 0 -> xyz=-38.333333333333336 51.666666666666664 23.7 rpy=0 0 0
- joint j_bld_36: origin xyz=-21.666666666666664 -51.666666666666664 16.15 rpy=0 0 0 -> xyz=-21.666666666666664 -51.666666666666664 21.25 rpy=0 0 0
- joint j_bld_37: origin xyz=-21.666666666666664 -45.0 18.45 rpy=0 0 0 -> xyz=-21.666666666666664 -45.0 17.4 rpy=0 0 0
- joint j_bld_38: origin xyz=-21.666666666666664 -38.333333333333336 16.0 rpy=0 0 0 -> xyz=-21.666666666666664 -38.333333333333336 17.1 rpy=0 0 0
- joint j_bld_39: origin xyz=-15.0 -51.666666666666664 17.85 rpy=0 0 0 -> xyz=-15.0 -51.666666666666664 19.9 rpy=0 0 0
- joint j_bld_4: origin xyz=-45.0 -45.0 15.55 rpy=0 0 0 -> xyz=-45.0 -45.0 15.4 rpy=0 0 0
- joint j_bld_40: origin xyz=-15.0 -45.0 19.25 rpy=0 0 0 -> xyz=-15.0 -45.0 21.6 rpy=0 0 0
- joint j_bld_41: origin xyz=-15.0 -38.333333333333336 22.35 rpy=0 0 0 -> xyz=-15.0 -38.333333333333336 18.25 rpy=0 0 0
- joint j_bld_42: origin xyz=-8.333333333333332 -51.666666666666664 23.4 rpy=0 0 0 -> xyz=-8.333333333333332 -51.666666666666664 21.85 rpy=0 0 0
- joint j_bld_43: origin xyz=-8.333333333333332 -45.0 20.7 rpy=0 0 0 -> xyz=-8.333333333333332 -45.0 19.2 rpy=0 0 0
- joint j_bld_44: origin xyz=-8.333333333333332 -38.333333333333336 22.0 rpy=0 0 0 -> xyz=-8.333333333333332 -38.333333333333336 19.35 rpy=0 0 0
- joint j_bld_45: origin xyz=-21.666666666666664 -21.666666666666664 23.4 rpy=0 0 0 -> xyz=-21.666666666666664 -21.666666666666664 21.95 rpy=0 0 0
- joint j_bld_46: origin xyz=-21.666666666666664 -15.0 21.1 rpy=0 0 0 -> xyz=-21.666666666666664 -15.0 21.6 rpy=0 0 0
- joint j_bld_47: origin xyz=-21.666666666666664 -8.333333333333332 17.6 rpy=0 0 0 -> xyz=-21.666666666666664 -8.333333333333332 19.35 rpy=0 0 0
- joint j_bld_48: origin xyz=-15.0 -21.666666666666664 16.0 rpy=0 0 0 -> xyz=-15.0 -21.666666666666664 19.6 rpy=0 0 0
- joint j_bld_49: origin xyz=-15.0 -15.0 23.15 rpy=0 0 0 -> xyz=-15.0 -15.0 22.65 rpy=0 0 0
- joint j_bld_5: origin xyz=-45.0 -38.333333333333336 16.85 rpy=0 0 0 -> xyz=-45.0 -38.333333333333336 23.05 rpy=0 0 0
- joint j_bld_50: origin xyz=-15.0 -8.333333333333332 15.45 rpy=0 0 0 -> xyz=-15.0 -8.333333333333332 16.45 rpy=0 0 0
- joint j_bld_51: origin xyz=-8.333333333333332 -21.666666666666664 20.5 rpy=0 0 0 -> xyz=-8.333333333333332 -21.666666666666664 19.05 rpy=0 0 0
- joint j_bld_52: origin xyz=-8.333333333333332 -15.0 24.75 rpy=0 0 0 -> xyz=-8.333333333333332 -15.0 24.15 rpy=0 0 0
- joint j_bld_53: origin xyz=-8.333333333333332 -8.333333333333332 21.5 rpy=0 0 0 -> xyz=-8.333333333333332 -8.333333333333332 18.55 rpy=0 0 0
- joint j_bld_54: origin xyz=-21.666666666666664 8.333333333333334 20.45 rpy=0 0 0 -> xyz=-21.666666666666664 8.333333333333334 15.45 rpy=0 0 0
- joint j_bld_55: origin xyz=-21.666666666666664 15.0 18.25 rpy=0 0 0 -> xyz=-21.666666666666664 15.0 24.85 rpy=0 0 0
- joint j_bld_56: origin xyz=-21.666666666666664 21.666666666666668 17.4 rpy=0 0 0 -> xyz=-21.666666666666664 21.666666666666668 15.4 rpy=0 0 0
- joint j_bld_57: origin xyz=-15.0 8.333333333333334 16.6 rpy=0 0 0 -> xyz=-15.0 8.333333333333334 22.55 rpy=0 0 0
- joint j_bld_58: origin xyz=-15.0 15.0 17.75 rpy=0 0 0 -> xyz=-15.0 15.0 20.1 rpy=0 0 0
- joint j_bld_59: origin xyz=-15.0 21.666666666666668 23.05 rpy=0 0 0 -> xyz=-15.0 21.666666666666668 19.2 rpy=0 0 0
- joint j_bld_6: origin xyz=-38.333333333333336 -51.666666666666664 23.65 rpy=0 0 0 -> xyz=-38.333333333333336 -51.666666666666664 21.05 rpy=0 0 0
- joint j_bld_60: origin xyz=-8.333333333333332 8.333333333333334 15.55 rpy=0 0 0 -> xyz=-8.333333333333332 8.333333333333334 18.7 rpy=0 0 0
- joint j_bld_61: origin xyz=-8.333333333333332 15.0 23.9 rpy=0 0 0 -> xyz=-8.333333333333332 15.0 22.1 rpy=0 0 0
- joint j_bld_62: origin xyz=-8.333333333333332 21.666666666666668 23.5 rpy=0 0 0 -> xyz=-8.333333333333332 21.666666666666668 17.9 rpy=0 0 0
- joint j_bld_63: origin xyz=-21.666666666666664 38.333333333333336 23.85 rpy=0 0 0 -> xyz=-21.666666666666664 38.333333333333336 20.2 rpy=0 0 0
- joint j_bld_64: origin xyz=-21.666666666666664 45.0 24.8 rpy=0 0 0 -> xyz=-21.666666666666664 45.0 16.15 rpy=0 0 0
- joint j_bld_65: origin xyz=-21.666666666666664 51.666666666666664 23.65 rpy=0 0 0 -> xyz=-21.666666666666664 51.666666666666664 20.8 rpy=0 0 0
- joint j_bld_66: origin xyz=-15.0 38.333333333333336 16.4 rpy=0 0 0 -> xyz=-15.0 38.333333333333336 15.8 rpy=0 0 0
- joint j_bld_67: origin xyz=-15.0 45.0 19.75 rpy=0 0 0 -> xyz=-15.0 45.0 22.1 rpy=0 0 0
- joint j_bld_68: origin xyz=-15.0 51.666666666666664 15.9 rpy=0 0 0 -> xyz=-15.0 51.666666666666664 23.65 rpy=0 0 0
- joint j_bld_69: origin xyz=-8.333333333333332 38.333333333333336 15.6 rpy=0 0 0 -> xyz=-8.333333333333332 38.333333333333336 20.75 rpy=0 0 0
- joint j_bld_7: origin xyz=-38.333333333333336 -45.0 20.65 rpy=0 0 0 -> xyz=-38.333333333333336 -45.0 18.8 rpy=0 0 0
- joint j_bld_70: origin xyz=-8.333333333333332 45.0 21.15 rpy=0 0 0 -> xyz=-8.333333333333332 45.0 18.4 rpy=0 0 0
- joint j_bld_71: origin xyz=-8.333333333333332 51.666666666666664 15.4 rpy=0 0 0 -> xyz=-8.333333333333332 51.666666666666664 23.2 rpy=0 0 0
- joint j_bld_72: origin xyz=8.333333333333334 -51.666666666666664 24.8 rpy=0 0 0 -> xyz=8.333333333333334 -51.666666666666664 22.3 rpy=0 0 0
- joint j_bld_73: origin xyz=8.333333333333334 -45.0 20.7 rpy=0 0 0 -> xyz=8.333333333333334 -45.0 15.45 rpy=0 0 0
- joint j_bld_74: origin xyz=8.333333333333334 -38.333333333333336 17.65 rpy=0 0 0 -> xyz=8.333333333333334 -38.333333333333336 23.2 rpy=0 0 0
- joint j_bld_75: origin xyz=15.0 -51.666666666666664 20.15 rpy=0 0 0 -> xyz=15.0 -51.666666666666664 23.2 rpy=0 0 0
- joint j_bld_76: origin xyz=15.0 -45.0 22.65 rpy=0 0 0 -> xyz=15.0 -45.0 21.45 rpy=0 0 0
- joint j_bld_77: origin xyz=15.0 -38.333333333333336 21.45 rpy=0 0 0 -> xyz=15.0 -38.333333333333336 21.85 rpy=0 0 0
- joint j_bld_78: origin xyz=21.666666666666668 -51.666666666666664 22.2 rpy=0 0 0 -> xyz=21.666666666666668 -51.666666666666664 20.3 rpy=0 0 0
- joint j_bld_79: origin xyz=21.666666666666668 -45.0 21.7 rpy=0 0 0 -> xyz=21.666666666666668 -45.0 17.9 rpy=0 0 0
- joint j_bld_8: origin xyz=-38.333333333333336 -38.333333333333336 24.8 rpy=0 0 0 -> xyz=-38.333333333333336 -38.333333333333336 15.4 rpy=0 0 0
- joint j_bld_80: origin xyz=21.666666666666668 -38.333333333333336 18.25 rpy=0 0 0 -> xyz=21.666666666666668 -38.333333333333336 21.55 rpy=0 0 0
- joint j_bld_81: origin xyz=8.333333333333334 -21.666666666666664 15.5 rpy=0 0 0 -> xyz=8.333333333333334 -21.666666666666664 24.45 rpy=0 0 0
- joint j_bld_82: origin xyz=8.333333333333334 -15.0 22.45 rpy=0 0 0 -> xyz=8.333333333333334 -15.0 18.35 rpy=0 0 0
- joint j_bld_83: origin xyz=8.333333333333334 -8.333333333333332 20.4 rpy=0 0 0 -> xyz=8.333333333333334 -8.333333333333332 18.45 rpy=0 0 0
- joint j_bld_84: origin xyz=15.0 -21.666666666666664 20.2 rpy=0 0 0 -> xyz=15.0 -21.666666666666664 18.5 rpy=0 0 0
- joint j_bld_85: origin xyz=15.0 -15.0 17.95 rpy=0 0 0 -> xyz=15.0 -15.0 22.9 rpy=0 0 0
- joint j_bld_86: origin xyz=15.0 -8.333333333333332 17.45 rpy=0 0 0 -> xyz=15.0 -8.333333333333332 17.25 rpy=0 0 0
- joint j_bld_87: origin xyz=21.666666666666668 -21.666666666666664 21.2 rpy=0 0 0 -> xyz=21.666666666666668 -21.666666666666664 23.25 rpy=0 0 0
- joint j_bld_88: origin xyz=21.666666666666668 -15.0 23.4 rpy=0 0 0 -> xyz=21.666666666666668 -15.0 22.95 rpy=0 0 0
- joint j_bld_89: origin xyz=21.666666666666668 -8.333333333333332 23.95 rpy=0 0 0 -> xyz=21.666666666666668 -8.333333333333332 15.6 rpy=0 0 0
- joint j_bld_9: origin xyz=-51.666666666666664 -21.666666666666664 17.55 rpy=0 0 0 -> xyz=-51.666666666666664 -21.666666666666664 23.35 rpy=0 0 0
- joint j_bld_90: origin xyz=8.333333333333334 8.333333333333334 21.6 rpy=0 0 0 -> xyz=8.333333333333334 8.333333333333334 18.6 rpy=0 0 0
- joint j_bld_91: origin xyz=8.333333333333334 15.0 22.2 rpy=0 0 0 -> xyz=8.333333333333334 15.0 17.4 rpy=0 0 0
- joint j_bld_92: origin xyz=8.333333333333334 21.666666666666668 16.3 rpy=0 0 0 -> xyz=8.333333333333334 21.666666666666668 16.6 rpy=0 0 0
- joint j_bld_93: origin xyz=15.0 8.333333333333334 19.9 rpy=0 0 0 -> xyz=15.0 8.333333333333334 22.85 rpy=0 0 0
- joint j_bld_94: origin xyz=15.0 15.0 21.4 rpy=0 0 0 -> xyz=15.0 15.0 22.05 rpy=0 0 0
- joint j_bld_95: origin xyz=15.0 21.666666666666668 16.7 rpy=0 0 0 -> xyz=15.0 21.666666666666668 19.5 rpy=0 0 0
- joint j_bld_96: origin xyz=21.666666666666668 8.333333333333334 19.85 rpy=0 0 0 -> xyz=21.666666666666668 8.333333333333334 18.45 rpy=0 0 0
- joint j_bld_97: origin xyz=21.666666666666668 15.0 17.55 rpy=0 0 0 -> xyz=21.666666666666668 15.0 24.45 rpy=0 0 0
- joint j_bld_98: origin xyz=21.666666666666668 21.666666666666668 16.4 rpy=0 0 0 -> xyz=21.666666666666668 21.666666666666668 17.7 rpy=0 0 0
- joint j_bld_99: origin xyz=8.333333333333334 38.333333333333336 18.9 rpy=0 0 0 -> xyz=8.333333333333334 38.333333333333336 23.0 rpy=0 0 0
